Commit message: Updated files to account for series of tests

File: urdf/vantage.urdf (robot description, URDF)
Before this commit: robot cartographer_backpack_3d, 3 links, 2 joints
Links:
- removed link 3dm_gx5_15
- removed link base_link
- removed link os1
- added link vantage
- added link vantage_2; visual box size=0.06 0.04 0.02
Joints:
- removed joint imu_link_joint
- removed joint os1_link_joint
- added joint vantage_joint: type fixed, parent vantage, child vantage_2, origin xyz=-0.0788 -0.0628 -0.4120 rpy=0.0020071 -0.0019928 0.007152
