Commit message: Preparing cartographer launch file and urdf

File: urdf/2_ouster_backpack.urdf (robot description, URDF)
Before this commit: robot cartographer_backpack_3d, 4 links, 3 joints
Links:
- removed link os1
- added link os1_1; visual cylinder length=0.07 radius=0.05
Joints:
- joint os1_link_joint: child os1 -> os1_1

Commit message: Updated launch and urdf files for Gene's ouster driver

File: urdf/2_ouster_backpack.urdf (robot description, URDF)
Before this commit: robot cartographer_backpack_3d, 4 links, 3 joints
Links:
- removed link os1_1
- removed link os1_2
- added link ouster_1/os1_lidar; visual cylinder length=0.07 radius=0.05
- added link ouster_2/os1_lidar; visual cylinder length=0.07 radius=0.05
Joints:
- joint os1_2_link_joint: child os1_2 -> ouster_2/os1_lidar; origin xyz=0.0 0.17145 -0.060325 rpy=1.5708, 0.0 0.0 -> xyz=0.0 0.17145 -0.060325 rpy=-1.5708 0.0 3.14159
- joint os1_link_joint: child os1_1 -> ouster_1/os1_lidar; origin xyz=0.0 0. 0.07 rpy=0.0 0.0 0.0 -> xyz=0.0 0. 0.07 rpy=0.0 0.0 3.14159

Commit message: changes for cart test

File: urdf/2_ouster_backpack.urdf (robot description, URDF)
Before this commit: robot cartographer_backpack_3d, 5 links, 4 joints
Links:
- removed link ouster_2/os1_lidar
- removed link servo
- added link v/os1_lidar; visual cylinder length=0.07 radius=0.05
Joints:
- removed joint saurav_link_joint
