Commit message: update from rig

File: shakeeb_launch/li_pkg-master/configs/qav500.urdf (robot description, URDF)
Before this commit: robot cartographer_backpack_3d, 5 links, 4 joints
Links:
- removed link h/os1_lidar
- removed link imu_link
- removed link servo
- removed link v/os1_lidar
- added link gx5_link; visual box size=0.06 0.04 0.02
- added link os1_lidar; visual cylinder length=0.07 radius=0.05
Joints:
- removed joint os1_2_link_joint
- removed joint saurav_link_joint
- joint imu_link_joint: child imu_link -> gx5_link; origin xyz=0 0 0 rpy=3.1416 0 1.5708 -> xyz=0 0 0 rpy=0 0 1.57
- joint os1_link_joint: child h/os1_lidar -> os1_lidar; origin xyz=0.0 0. 0.07 rpy=0.0 0.0 3.14159 -> xyz=0 0 -0.03 rpy=3.14 0 3.14

File: urdf/ouster_backpack.urdf (robot description, URDF)
Before this commit: robot cartographer_backpack_3d, 3 links, 2 joints
Links:
- removed link 3dm_gx5_15
- added link imu_link; visual box size=0.06 0.04 0.02
Joints:
- joint imu_link_joint: child 3dm_gx5_15 -> imu_link
